File: esp32-mp3-board/esp32-mp3-board.kicad_pcb (KiCad board)
At the start: 2 copper layers, 0 parts

Commit message: add esp32-mp3-board
Parts:
- added C1: 10uF, OPL_Capacitor:C0603, F.Cu at (142.4, 110.1)
- added C10: 220pF, OPL_Capacitor:C0603, F.Cu at (170.3, 99.2)
- added C2: 10uF, OPL_Capacitor:C0603, F.Cu at (164.2, 105.7)
- added C3: 10uF, OPL_Capacitor:C0603, F.Cu at (167.3, 88.8)
- added C4: 0.1uF, OPL_Capacitor:C0603, F.Cu at (163.4, 92.5)
- added C5: 10uF, OPL_Capacitor:C0603, F.Cu at (164.2, 109.3)
- added C6: 1uF, OPL_Capacitor:C0603, F.Cu at (161.3, 112.1)
- added C7: 10uF, OPL_Capacitor:C0603, F.Cu at (135.6, 77.0)
- added C8: 1uF, OPL_Capacitor:C0603, F.Cu at (125.7, 86.9)
- added C9: 220pF, OPL_Capacitor:C0603, F.Cu at (170.3, 88.8)
- added D1: D_Schottky, Diode_SMD:D_SOD-123, F.Cu at (149.7, 104.5)
- added D2: LED, LED_SMD:LED_0603_1608Metric, F.Cu at (149.0, 98.7)
- added D3: WS2812S, LED_SMD:LED_WS2812_PLCC6_5.0x5.0mm_P1.6mm, F.Cu at (165.0, 120.0)
- added D4: WS2812S, LED_SMD:LED_WS2812_PLCC6_5.0x5.0mm_P1.6mm, F.Cu at (128.5, 67.1)
- added D5: 1N4148, OPL_Discrete_Semiconductor:SOD-123, F.Cu at (144.5, 104.5)
- added J1: USB_C_Receptacle_USB2.0, Connector_USB:USB_C_Receptacle_Palconn_UTC16-G, F.Cu at (146.8, 119.1)
- added J2: Conn_01x02, OPL_Connector:H2-2.54, F.Cu at (136.4, 121.4)
- added J3: UART, OPL_Connector:H6-2.54, F.Cu at (118.6, 82.0)
- added J4: TOUCH, OPL_Connector:H3-2.54, F.Cu at (118.6, 109.5)
- added J5: Conn_01x04, OPL_Connector:H4-2.54, F.Cu at (118.6, 97.7)
- added L1: SMD-FERRITE, OPL_Resistor:R0603, F.Cu at (167.9, 95.4)
- added L2: SMD-FERRITE, OPL_Resistor:R0603, F.Cu at (167.9, 92.5)
- added Q1: S9013, Package_TO_SOT_SMD:TSOT-23, F.Cu at (130.9, 88.4)
- added Q2: S9013, Package_TO_SOT_SMD:TSOT-23, F.Cu at (130.8, 82.3)
- added R1: 100k, OPL_Resistor:R0603, F.Cu at (151.6, 110.1)
- added R10: 5.1K, OPL_Resistor:R0603, F.Cu at (145.5, 110.1)
- added R11: 5.1K, OPL_Resistor:R0603, F.Cu at (148.6, 110.1)
- added R2: 100k, OPL_Resistor:R0603, F.Cu at (159.5, 104.4)
- added R3: 1M, OPL_Resistor:R0603, F.Cu at (163.4, 95.4)
- added R4: 10k, OPL_Resistor:R0603, F.Cu at (125.7, 89.7)
- added R5: 10k, OPL_Resistor:R0603, F.Cu at (125.7, 81.3)
- added R6: 10k, OPL_Resistor:R0603, F.Cu at (125.7, 84.1)
- added R7: 100, OPL_Resistor:R0603, F.Cu at (157.6, 116.0)
- added R9: 1k, OPL_Resistor:R0603, F.Cu at (144.3, 98.7)
- added REF**: MountingHole_3.2mm_M3, MountingHole:MountingHole_3.2mm_M3, F.Cu at (172.8, 67.6)
- added REF**: MountingHole_3.2mm_M3, MountingHole:MountingHole_3.2mm_M3, F.Cu at (120.8, 67.6)
- added REF**: MountingHole_3.2mm_M3, MountingHole:MountingHole_3.2mm_M3, F.Cu at (120.8, 119.6)
- added REF**: MountingHole_3.2mm_M3, MountingHole:MountingHole_3.2mm_M3, F.Cu at (172.8, 119.6)
- added SW1: SW_PUSH, Button_Switch_SMD:SW_Push_1P1T_NO_CK_KMR2, F.Cu at (129.0, 120.8)
- added U1: AP2112K-3.3, Package_TO_SOT_SMD:SOT-23-5, F.Cu at (159.5, 108.6)
- added U2: ESP32-WROOM-32, RF_Module:ESP32-WROOM-32, F.Cu at (147.1, 84.6)
- added U3: MAX98357AETE+T, open-automation:MAX98357A, F.Cu at (161.9, 87.2)
- added X1: Conn_01x02, OPL_Connector:H2-2.54, F.Cu at (174.9, 98.3)
- added X2: Conn_01x02, OPL_Connector:H2-2.54, F.Cu at (174.9, 89.5)
Routing:
- net GND: track 0.00 -> 210.7 mm, vias 0 -> 107
- net +3V3: track 0.00 -> 180.6 mm, vias 0 -> 7
- net Net-(D3-Pad1): track 0.00 -> 87.9 mm
- net /VDD: track 0.00 -> 87.8 mm, vias 0 -> 6
- net /RESET: track 0.00 -> 70.5 mm, vias 0 -> 2
- net /SCL: track 0.00 -> 55.9 mm, vias 0 -> 3
- net /SDA: track 0.00 -> 53.8 mm, vias 0 -> 3
- net /T9: track 0.00 -> 40.4 mm, vias 0 -> 2
- net /T8: track 0.00 -> 39.1 mm, vias 0 -> 2
- net /RX: track 0.00 -> 38.2 mm, vias 0 -> 2
- net /TX: track 0.00 -> 37.7 mm, vias 0 -> 2
- net /DTR: track 0.00 -> 36.6 mm, vias 0 -> 2
- net /IO4: track 0.00 -> 36.3 mm, vias 0 -> 2
- net VBUS: track 0.00 -> 35.0 mm, vias 0 -> 2
- net /T7: track 0.00 -> 31.9 mm, vias 0 -> 4
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- added copper zone on B.Cu, net GND
- added copper zone on F.Cu, net GND
Other:
- board outline added: 60 x 60 mm
- net class Bold added: clearance 0.2, trace_width 0.4, via_dia 0.6, via_drill 0.3
- board text added: "3V3"
- board text added: "AUDIO OUT"
- board text added: "CTS"
- board text added: "ConnectedDoll ver.0.1"
- board text added: "DTR"
- board text added: "GND"
- board text added: "I2C"
- board text added: "POWER"
- board text added: "RESET"
- board text added: "RX"
- board text added: "SCL"
- board text added: "SDA"
- board text added: "T7"
- board text added: "T8"
- board text added: "T9"
- board text added: "TOUCH"
- board text added: "TX"
- board text added: "UART"

Commit message: RTS追加 CTS回路修正
Connections:
- J3 pad 5: /CTS -> /RTS
- Q2 pad 2: /RESET -> /RTS
- R5 pad 2: /RESET -> /RTS
Routing:
- net /RTS: track 0.00 -> 11.1 mm, vias 0 -> 1
